File: board/romprogrammer.kicad_pcb (KiCad board)
At the start: 2 copper layers, 5 parts, among them U1 ARDUINO_NANO_V3, U2 74HC595, U3 74HC595, U4 74HC595, U5 SST39SF020

Commit message: fo
Parts:
- moved U1 80.8 mm to (52.7, 33.7)
- moved U2 80.8 mm to (41.9, 76.8)
- moved U3 80.8 mm to (66.7, 100.3)
- moved U4 80.8 mm to (73.7, 71.8)
- moved U5 80.8 mm to (57.8, 71.8)

Commit message: updates
Routing:
- net GND: track 248.6 -> 141.9 mm
Changed lines of the file:
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@@
   (general
     (links 53)
-    (no_connects 2)
+    (no_connects 3)
     (area 9.295001 13.81 83.820001 107.950001)
     (thickness 1.6)
     (drawings 6)
-    (tracks 250)
+    (tracks 223)
     (zones 0)
     (modules 5)
@@
   (page A4 portrait)
   (layers
-    (0 F.Cu signal)
+    (0 F.Cu signal hide)
     (31 B.Cu signal)
     (32 B.Adhes user)
@@
   )
   (segment (start 38.1 26.67) (end 38.1 30.48) (width 0.5) (layer F.Cu) (net 3))
+  (segment (start 38.1 30.48) (end 43.18 35.56) (width 0.5) (layer F.Cu) (net 3))
   (segment (start 43.18 35.56) (end 43.18 41.91) (width 0.5) (layer F.Cu) (net 3))
-  (segment (start 38.1 30.48) (end 43.18 35.56) (width 0.5) (layer F.Cu) (net 3))
   (segment (start 57.785 96.52) (end 57.785 97.79) (width 0.5) (layer F.Cu) (net 3))
   (segment (start 67.945 102.235) (end 67.945 104.14) (width 0.5) (layer F.Cu) (net 3))
@@
   (segment (start 38.1 36.83) (end 40.005 38.735) (width 0.5) (layer B.Cu) (net 3))
   (segment (start 43.18 41.91) (end 43.18 42.545) (width 0.5) (layer B.Cu) (net 3))
-  (segment (start 43.18 42.545) (end 43.815 43.18) (width 0.5) (layer B.Cu) (net 3))
-  (segment (start 45.085 67.31) (end 45.72 67.945) (width 0.5) (layer B.Cu) (net 3))
-  (segment (start 45.085 58.42) (end 45.085 67.31) (width 0.5) (layer B.Cu) (net 3))
-  (segment (start 43.18 56.515) (end 45.085 58.42) (width 0.5) (layer B.Cu) (net 3))
-  (segment (start 43.18 49.53) (end 43.18 56.515) (width 0.5) (layer B.Cu) (net 3))
-  (segment (start 43.815 48.895) (end 43.18 49.53) (width 0.5) (layer B.Cu) (net 3))
-  (segment (start 43.815 43.18) (end 43.815 48.895) (width 0.5) (layer B.Cu) (net 3))
-  (segment (start 74.295 79.375) (end 74.295 82.55) (width 0.5) (layer B.Cu) (net 3))
-  (segment (start 59.055 98.425) (end 57.785 97.155) (width 0.5) (layer B.Cu) (net 3))
-  (segment (start 76.2 98.425) (end 59.055 98.425) (width 0.5) (layer B.Cu) (net 3))
-  (segment (start 77.47 97.155) (end 76.2 98.425) (width 0.5) (layer B.Cu) (net 3))
-  (segment (start 77.47 95.885) (end 77.47 97.155) (width 0.5) (layer B.Cu) (net 3))
-  (segment (start 75.565 93.98) (end 77.47 95.885) (width 0.5) (layer B.Cu) (net 3))
-  (segment (start 75.565 83.82) (end 75.565 93.98) (width 0.5) (layer B.Cu) (net 3))
-  (segment (start 74.295 82.55) (end 75.565 83.82) (width 0.5) (layer B.Cu) (net 3))
-  (segment (start 57.785 97.155) (end 57.785 96.52) (width 0.5) (layer B.Cu) (net 3))
-  (segment (start 65.405 52.705) (end 71.12 52.705) (width 0.5) (layer B.Cu) (net 3))
-  (segment (start 73.025 80.645) (end 69.85 80.645) (width 0.5) (layer B.Cu) (net 3))
-  (segment (start 74.295 79.375) (end 73.025 80.645) (width 0.5) (layer B.Cu) (net 3))
-  (segment (start 74.295 73.66) (end 74.295 79.375) (width 0.5) (layer B.Cu) (net 3))
-  (segment (start 73.025 72.39) (end 74.295 73.66) (width 0.5) (layer B.Cu) (net 3))
-  (segment (start 73.025 69.215) (end 73.025 72.39) (width 0.5) (layer B.Cu) (net 3))
-  (segment (start 71.755 67.945) (end 73.025 69.215) (width 0.5) (layer B.Cu) (net 3))
-  (segment (start 71.755 59.69) (end 71.755 67.945) (width 0.5) (layer B.Cu) (net 3))
-  (segment (start 72.39 59.055) (end 71.755 59.69) (width 0.5) (layer B.Cu) (net 3))
-  (segment (start 72.39 53.975) (end 72.39 59.055) (width 0.5) (layer B.Cu) (net 3))
-  (segment (start 71.12 52.705) (end 72.39 53.975) (width 0.5) (layer B.Cu) (net 3))
   (segment (start 43.18 26.67) (end 43.18 25.4) (width 0.5) (layer B.Cu) (net 4))
   (segment (start 33.655 25.4) (end 33.655 38.735) (width 0.5) (layer B.Cu) (net 4))

Commit message: fixed board
Connections:
- U1 pad 1: (no net) -> Net-(U1-Pad1)
- U1 pad 16: (no net) -> Net-(U1-Pad16)
- U1 pad 17: (no net) -> Net-(U1-Pad17)
- U1 pad 18: (no net) -> Net-(U1-Pad18)
- U1 pad 19: (no net) -> Net-(U1-Pad19)
- U1 pad 2: (no net) -> Net-(U1-Pad2)
- U1 pad 22: (no net) -> Net-(U1-Pad22)
- U1 pad 23: (no net) -> Net-(U1-Pad23)
- U1 pad 24: (no net) -> Net-(U1-Pad24)
- U1 pad 25: (no net) -> Net-(U1-Pad25)
- U1 pad 26: (no net) -> Net-(U1-Pad26)
- U1 pad 28: (no net) -> Net-(U1-Pad28)
- U1 pad 3: (no net) -> Net-(U1-Pad3)
- U1 pad 30: (no net) -> Net-(U1-Pad30)
- U2 pad 15: (no net) -> Net-(U2-Pad15)
- U2 pad 9: (no net) -> Net-(U2-Pad9)
- U3 pad 15: (no net) -> Net-(U3-Pad15)
- U3 pad 5: (no net) -> Net-(U3-Pad5)
- U3 pad 6: (no net) -> Net-(U3-Pad6)
- U3 pad 7: (no net) -> Net-(U3-Pad7)
- U4 pad 15: (no net) -> Net-(U4-Pad15)
- U5 pad 1: (no net) -> Net-(U5-Pad1)
- U5 pad 22: VCC -> GND
Routing:
- net /RCLK: track 134.9 -> 137.1 mm
- net Net-(U3-Pad14): track 31.5 -> 30.4 mm
- net /SRCLK: track 128.2 -> 127.7 mm
Other:
- net class Default: clearance 0.5 -> 0.4; via_dia 0.6 -> 1.4; via_drill 0.4 -> 0.81
- rule trace_clearance: 0.5 -> 0.4
